File: Hardware/BattleBot_Motherboard/BattleBot_Motherboard.kicad_sch (KiCad schematic)
At the start: 11 parts, among them J1 Conn_01x04

Commit message: Make a 3d model of esp
Parts:
- added U1: ESP32-S2-WROVER, Espressif:ESP32-S2-WROVER, symbol Espressif:ESP32-S2-WROVER
Changed lines of the file:
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@@
     (pin "2")
+  )
+  (symbol (lib_id "Espressif:ESP32-S2-WROVER") (at 144.78 81.28 0) (unit 1)
+    (in_bom yes) (on_board yes) (fields_autoplaced)
+    (property "Reference" "U1" (id 0) (at 145.415 31.75 0))
+    (property "Value" "ESP32-S2-WROVER" (id 1) (at 145.415 34.29 0))
+    (property "Footprint" "Espressif:ESP32-S2-WROVER" (id 2) (at 144.78 129.54 0)
+      (effects (font (size 1.27 1.27)) hide)
+    )
+    (property "Datasheet" "https://www.espressif.com/sites/default/files/documentation/esp32-s2-wroom_esp32-s2-wroom-i_datasheet_en.pdf" (id 3) (at 144.78 81.28 0)
+      (effects (font (size 1.27 1.27)) hide)
+    )
+    (pin "1")
+    (pin "10")
+    (pin "11")
+    (pin "12")
+    (pin "13")
+    (pin "14")
+    (pin "15")
+    (pin "16")
+    (pin "17")
+    (pin "18")
+    (pin "19")
+    (pin "2")
+    (pin "20")
+    (pin "21")
+    (pin "22")
+    (pin "23")
+    (pin "24")
+    (pin "25")
+    (pin "26")
+    (pin "27")
+    (pin "28")
+    (pin "29")
+    (pin "3")
+    (pin "30")
+    (pin "31")
+    (pin "32")
+    (pin "33")
+    (pin "34")
+    (pin "35")
+    (pin "36")
+    (pin "37")
+    (pin "38")
+    (pin "39")
+    (pin "4")
+    (pin "40")
+    (pin "41")
+    (pin "42")
+    (pin "43")
+    (pin "5")
+    (pin "6")
+    (pin "7")
+    (pin "8")
+    (pin "9")
   )
   (symbol (lib_id "Device:R") (at 50.8 38.1 270) (unit 1)
@@
       (reference "R3") (unit 1) (value "220") (footprint "Resistor_THT:R_Axial_DIN0204_L3.6mm_D1.6mm_P5.08mm_Horizontal")
     )
+    (path "/afa121ea-3a3e-4391-ae30-44a18537c157"
+      (reference "U1") (unit 1) (value "ESP32-S2-WROVER") (footprint "Espressif:ESP32-S2-WROVER")
+    )
   )
