File: Hardware/BattleBot_Motherboard/BattleBot_Motherboard.kicad_pcb (KiCad board)
At the start: 2 copper layers, 30.7 x 39.4 mm, 11 parts, among them J1 Conn_01x04

Commit message: Make a 3d model of esp
Parts:
- added U1: ESP32-S2-WROVER, Espressif:ESP32-S2-WROVER, F.Cu at (119.4, 108.0)
Other:
- board size 30.7 x 39.4 mm -> 58.4 x 39.4 mm
